Commit message: controllers.yaml actualization

File: warthog_description/urdf/warthog.urdf.xacro (robot description, xacro)
@@ -1,95 +1,101 @@
 <?xml version="1.0"?>
 <robot name="warthog" xmlns:xacro="http://www.ros.org/wiki/xacro">
-  <xacro:property name="PI" value="3.1415926535897931"/>
-  <xacro:property name="wheel_radius" value="0.3" />
-  <xacro:property name="wheel_width" value="0.25" />
-  <xacro:property name="wheel_mass" value="15" />
-  <xacro:property name="wheel_to_track_ratio" value="0.5962" />
-  <xacro:property name="axle_x_offset" value="0.457367" />
-  <xacro:property name="axle_y_offset" value="0.0" />
-  <xacro:property name="axle_z_offset" value="-0.012977" />
-  <xacro:property name="diff_unit_length" value="1.34" />
-  <xacro:property name="diff_unit_width" value="0.28" />
-  <xacro:property name="diff_unit_height" value="0.63"/>
-  <xacro:property name="diff_unit_mass" value="50" />
-  <xacro:property name="diff_unit_offset_x" value="0.00" />
-  <xacro:property name="diff_unit_offset_y" value="0.56821" />
-  <xacro:property name="diff_unit_offset_z" value="0.0" />
-  <xacro:property name="chassis_length" value="1.35" />
-  <xacro:property name="chassis_width" value="0.70" />
-  <xacro:property name="chassis_height" value="0.30" />
-  <xacro:property name="chassis_mass" value="100" />
-  <xacro:property name="dummy_inertia" value="1e-09"/>
-  <!--
-    Optional paint colors.
-    Available colors:
-      - yellow (default)
-      - orange
-      - olive
-      - sand
-  -->
-  <xacro:macro name="wheel_inertia" params="m r h">
-    <inertia ixx="${m*(3*r*r+h*h)/12}" ixy="0" ixz="0"
-             iyy="${m*r*r/2}" iyz="0"
-             izz="${m*(3*r*r+h*h)/12}" />
-  </xacro:macro>
-  <xacro:macro name="box_inertia" params="m x y z">
-    <inertia ixx="${m*(y*y+z*z)/12}" ixy="0" ixz="0"
-             iyy="${m*(x*x+z*z)/12}" iyz="0"
-             izz="${m*(x*x+z*z)/12}" />
-  </xacro:macro>
-  <material name="dark_grey"><color rgba="0.2 0.2 0.2 1.0" /></material>
-  <material name="light_grey"><color rgba="0.4 0.4 0.4 1.0" /></material>
-  <material name="yellow"><color rgba="0.95 0.816 0.082 1.0" /></material>
-  <material name="black"><color rgba="0.15 0.15 0.15 1.0" /></material>
-  <material name="white"><color rgba="0.9 0.9 0.9 1.0" /></material>
-  <material name="red"><color rgba="0.9 0.0 0.0 1.0" /></material>
-  <xacro:macro name="wheel" params="prefix side *joint_pose">
-    <link name="${prefix}_${side}_wheel_link">
-      <inertial>
-        <origin xyz="0 0 0" rpy="0 0 0" />
-        <mass value="${wheel_mass}" />
-        <xacro:wheel_inertia m="${wheel_mass}" r="${wheel_radius}" h="${wheel_width}" />
-      </inertial>
-      <visual>
-        <origin xyz="0 0 0" rpy="0 0 ${PI/2}"/>
-        <geometry>
-          <mesh filename="package://warthog_description/meshes/wheel.stl" />
-        </geometry>
-        <material name="dark_grey" />
-      </visual>
-      <collision>
-        <origin xyz="0 0 0" rpy="${PI/2} 0 0"/>
-        <geometry>
-          <cylinder radius="${wheel_radius}" length="${wheel_width}"/>
-        </geometry>
-      </collision>
-    </link>
-    <joint name="${prefix}_${side}_wheel_joint" type="continuous">
-      <parent link="${side}_diff_unit_link"/>
-      <child link="${prefix}_${side}_wheel_link"/>
-      <xacro:insert_block name="joint_pose" />
-      <axis xyz="0 1 0"/>
-    </joint>
-    <gazebo reference="${prefix}_${side}_wheel_link">
-      <selfCollide>false</selfCollide>
-      <mu1>0.5</mu1>
-      <mu2>0.5</mu2>
-      <kp value="10000000.0" />
-      <kd value="1.0" />
-      <fdir1 value="1 0 0" />
-      <material>Gazebo/DarkGrey</material>
-    </gazebo>
-    <transmission name="${prefix}_${side}_wheel_trans">
-      <type>transmission_interface/SimpleTransmission</type>
-      <joint name="${prefix}_${side}_wheel_joint">
-        <hardwareInterface>hardware_interface/VelocityJointInterface</hardwareInterface>
-      </joint>
-      <actuator name="${prefix}_${side}_actuator">
-        <hardwareInterface>hardware_interface/VelocityJointInterface</hardwareInterface>
-        <mechanicalReduction>1</mechanicalReduction>
-      </actuator>
-    </transmission>
-  </xacro:macro>
+    <xacro:property name="PI" value="3.1415926535897931"/>
+    <xacro:property name="wheel_radius" value="0.3" />
+    <xacro:property name="wheel_width" value="0.25" />
+    <xacro:property name="wheel_mass" value="15" />
+    <xacro:property name="wheel_to_track_ratio" value="0.5962" />
+    <xacro:property name="axle_x_offset" value="0.457367" />
+    <xacro:property name="axle_y_offset" value="0.0" />
+    <xacro:property name="axle_z_offset" value="-0.012977" />
+    <xacro:property name="diff_unit_length" value="1.34" />
+    <xacro:property name="diff_unit_width" value="0.28" />
+    <xacro:property name="diff_unit_height" value="0.63"/>
+    <xacro:property name="diff_unit_mass" value="50" />
+    <xacro:property name="diff_unit_offset_x" value="0.00" />
+    <xacro:property name="diff_unit_offset_y" value="0.56821" />
+    <xacro:property name="diff_unit_offset_z" value="0.0" />
+    <xacro:property name="chassis_length" value="1.35" />
+    <xacro:property name="chassis_width" value="0.70" />
+    <xacro:property name="chassis_height" value="0.30" />
+    <xacro:property name="chassis_mass" value="100" />
+    <xacro:property name="dummy_inertia" value="1e-09"/>
+    <!--
+        Optional paint colors.
+        Available colors:
+        - yellow (default)
+        - orange
+        - olive
+        - sand
+    -->
+    <xacro:macro name="wheel_inertia" params="m r h">
+        <inertia ixx="${m*(3*r*r+h*h)/12}" ixy="0" ixz="0"
+                iyy="${m*r*r/2}" iyz="0"
+                izz="${m*(3*r*r+h*h)/12}" />
+    </xacro:macro>
+    <xacro:macro name="box_inertia" params="m x y z">
+        <inertia ixx="${m*(y*y+z*z)/12}" ixy="0" ixz="0"
+                iyy="${m*(x*x+z*z)/12}" iyz="0"
+                izz="${m*(x*x+z*z)/12}" />
+    </xacro:macro>
+    <material name="dark_grey"><color rgba="0.2 0.2 0.2 1.0" /></material>
+    <material name="light_grey"><color rgba="0.4 0.4 0.4 1.0" /></material>
+    <material name="yellow"><color rgba="0.95 0.816 0.082 1.0" /></material>
+    <material name="black"><color rgba="0.15 0.15 0.15 1.0" /></material>
+    <material name="white"><color rgba="0.9 0.9 0.9 1.0" /></material>
+    <material name="red"><color rgba="0.9 0.0 0.0 1.0" /></material>
+    <!-- ======================================================= -->
+    <!--                      Wheels                         -->
+    <!-- ======================================================= -->
+    <xacro:macro name="wheel" params="prefix side *joint_pose">
+        <link name="${prefix}_${side}_wheel_link">
+        <inertial>
+            <origin xyz="0 0 0" rpy="0 0 0" />
+            <mass value="${wheel_mass}" />
+            <xacro:wheel_inertia m="${wheel_mass}" r="${wheel_radius}" h="${wheel_width}" />
+        </inertial>
+        <visual>
+            <origin xyz="0 0 0" rpy="0 0 ${PI/2}"/>
+            <geometry>
+            <mesh filename="package://warthog_description/meshes/wheel.stl" />
+            </geometry>
+            <material name="dark_grey" />
+        </visual>
+        <collision>
+            <origin xyz="0 0 0" rpy="${PI/2} 0 0"/>
+            <geometry>
+            <cylinder radius="${wheel_radius}" length="${wheel_width}"/>
+            </geometry>
+        </collision>
+        </link>
+        <joint name="${prefix}_${side}_wheel_joint" type="continuous">
+            <parent link="${side}_diff_unit_link"/>
+            <child link="${prefix}_${side}_wheel_link"/>
+            <xacro:insert_block name="joint_pose" />
+            <axis xyz="0 1 0"/>
+        </joint>
+        <gazebo reference="${prefix}_${side}_wheel_link">
+            <selfCollide>false</selfCollide>
+            <mu1>0.5</mu1>
+            <mu2>0.5</mu2>
+            <kp value="10000000.0" />
+            <kd value="1.0" />
+            <fdir1 value="1 0 0" />
+            <material>Gazebo/DarkGrey</material>
+        </gazebo>
+        <transmission name="${prefix}_${side}_wheel_trans">
+            <type>transmission_interface/SimpleTransmission</type>
+            <joint name="${prefix}_${side}_wheel_joint">
+                <hardwareInterface>hardware_interface/VelocityJointInterface</hardwareInterface>
+            </joint>
+            <actuator name="${prefix}_${side}_actuator">
+                <hardwareInterface>hardware_interface/VelocityJointInterface</hardwareInterface>
+                <mechanicalReduction>1</mechanicalReduction>
+            </actuator>
+        </transmission>
+    </xacro:macro>
+    <!-- ======================================================= -->
+    <!--                       Tracks                          -->
+    <!-- ======================================================= -->
     <xacro:macro name="track" params="prefix side *joint_pose">
         <link name="${prefix}_${side}_track_link">

Commit message: gz working and rviz not

File: warthog_description/urdf/warthog.urdf.xacro (robot description, xacro)
@@ -58,5 +58,5 @@
             <origin xyz="0 0 0" rpy="0 0 ${PI/2}"/>
             <geometry>
-            <mesh filename="package://warthog_description/meshes/wheel.stl" />
+            <mesh filename="model://warthog_description/meshes/wheel.stl" />
             </geometry>
             <material name="dark_grey" />
@@ -103,5 +103,5 @@
             <origin xyz="0 0 0" rpy="0 0 0"/>
             <geometry>
-            <mesh filename="package://warthog_description/meshes/tracks.dae" />
+            <mesh filename="model://warthog_description/meshes/tracks.dae" />
             </geometry>
             <material name="dark_grey" />
@@ -110,5 +110,5 @@
             <origin xyz="0 0 0" rpy="0 0 0"/>
             <geometry>
-            <mesh filename="package://warthog_description/meshes/tracks_collision.stl" />
+            <mesh filename="model://warthog_description/meshes/tracks_collision.stl" />
             </geometry>
         </collision>
@@ -197,5 +197,5 @@
             <origin xyz="0 0 0" rpy="0 0 0"/>
             <geometry>
-                <mesh filename="package://warthog_description/meshes/chassis.stl" />
+                <mesh filename="model://warthog_description/meshes/chassis.stl" />
             </geometry>
             <material name="black"><color rgba="0.15 0.15 0.15 1.0" /></material>
@@ -204,5 +204,5 @@
             <origin xyz="0 0 0" rpy="0 0 0"/>
             <geometry>
-                <mesh filename="package://warthog_description/meshes/e-stop.stl" />
+                <mesh filename="model://warthog_description/meshes/e-stop.stl" />
             </geometry>
             <material name="red"><color rgba="0.9 0.0 0.0 1.0" /></material>
@@ -211,5 +211,5 @@
             <origin xyz="0 0 0" rpy="0 0 0"/>
             <geometry>
-                <mesh filename="package://warthog_description/meshes/chassis-collision.stl" />
+                <mesh filename="model://warthog_description/meshes/chassis-collision.stl" />
             </geometry>
         </collision>
@@ -223,5 +223,5 @@
             <origin xyz="0 0 0" rpy="0 0 0"/>
             <geometry>
-                <mesh filename="package://warthog_description/meshes/diff-link.stl" />
+                <mesh filename="model://warthog_description/meshes/diff-link.stl" />
             </geometry>
             <material name="light_grey" />
@@ -230,5 +230,5 @@
             <origin xyz="0 0 0" rpy="0 0 0"/>
             <geometry>
-                <mesh filename="package://warthog_description/meshes/susp-link.stl" />
+                <mesh filename="model://warthog_description/meshes/susp-link.stl" />
             </geometry>
             <material name="light_grey" />
@@ -237,5 +237,5 @@
             <origin xyz="0 0 0" rpy="0 0 0"/>
             <geometry>
-                <mesh filename="package://warthog_description/meshes/susp-link.stl" />
+                <mesh filename="model://warthog_description/meshes/susp-link.stl" />
             </geometry>
             <material name="light_grey" />
@@ -262,5 +262,5 @@
             <origin xyz="0 0 0" rpy="0 0 ${side*PI/2}"/>
             <geometry>
-            <mesh filename="package://warthog_description/meshes/rocker.stl" />
+            <mesh filename="model://warthog_description/meshes/rocker.stl" />
             </geometry>
             <material name="black"><color rgba="0.15 0.15 0.15 1.0" /></material>
@@ -269,5 +269,5 @@
             <origin xyz="0 0 0" rpy="0 0 ${side*PI/2}"/>
             <geometry>
-            <mesh filename="package://warthog_description/meshes/fenders.stl" />
+            <mesh filename="model://warthog_description/meshes/fenders.stl" />
             </geometry>
             <material name="yellow"><color rgba="0.95 0.816 0.082 1.0" /></material>
@@ -276,5 +276,5 @@
             <origin xyz="0 0 0" rpy="0 0 ${side*PI/2}"/>
             <geometry>
-            <mesh filename="package://warthog_description/meshes/fenders-collision.stl" />
+            <mesh filename="model://warthog_description/meshes/fenders-collision.stl" />
             </geometry>
         </collision>
@@ -300,5 +300,5 @@
         <visual>
             <geometry>
-            <mesh filename="package://warthog_description/meshes/buttons.stl"/>
+            <mesh filename="model://warthog_description/meshes/buttons.stl"/>
             </geometry>
             <material name="red"><color rgba="0.9 0.0 0.0 1.0" /></material>
@@ -324,5 +324,5 @@
                 <material name="light_grey" />
                 <geometry>
-                <mesh filename="package://warthog_description/meshes/antenna_${prefix}.stl"/>
+                <mesh filename="model://warthog_description/meshes/antenna_${prefix}.stl"/>
                 </geometry>
             </visual>
@@ -348,5 +348,5 @@
                 <material name="light_grey"/>
                 <geometry>
-                    <mesh filename="package://warthog_description/meshes/antenna_estop.stl"/>
+                    <mesh filename="model://warthog_description/meshes/antenna_estop.stl"/>
                 </geometry>
                 </visual>
@@ -372,5 +372,5 @@
                 <origin xyz="0 ${side*-0.029} 0" rpy="0 0 0"/>
                 <geometry>
-                    <mesh filename="package://warthog_description/meshes/light.stl" />
+                    <mesh filename="model://warthog_description/meshes/light.stl" />
                 </geometry>
                 <material name="white"><color rgba="0.9 0.9 0.9 1.0" /></material>
@@ -379,5 +379,5 @@
                 <origin xyz="0 ${side*-0.022} 0" rpy="0 0 0"/>
                 <geometry>
-                <mesh filename="package://warthog_description/meshes/light-collision.stl" />
+                <mesh filename="model://warthog_description/meshes/light-collision.stl" />
                 </geometry>
                 <material name="white"><color rgba="0.9 0.9 0.9 1.0" /></material>
@@ -406,5 +406,5 @@
                 <origin xyz="0 ${side*-0.029} 0" rpy="0 0 ${side*PI}"/>
                 <geometry>
-                <mesh filename="package://warthog_description/meshes/light.stl" />
+                <mesh filename="model://warthog_description/meshes/light.stl" />
                 </geometry>
                 <material name="red"><color rgba="0.9 0.0 0.0 1.0" /></material>
@@ -413,5 +413,5 @@
                 <origin xyz="0 ${side*-0.022} 0" rpy="0 0 ${side*PI}"/>
                 <geometry>
-                <mesh filename="package://warthog_description/meshes/light-collision.stl" />
+                <mesh filename="model://warthog_description/meshes/light-collision.stl" />
                 </geometry>
                 <material name="red"><color rgba="0.9 0.0 0.0 1.0" /></material>

Commit message: gz working and rviz working

File: warthog_description/urdf/warthog.urdf.xacro (robot description, xacro)
@@ -58,5 +58,5 @@
             <origin xyz="0 0 0" rpy="0 0 ${PI/2}"/>
             <geometry>
-            <mesh filename="model://warthog_description/meshes/wheel.stl" />
+            <mesh filename="package://warthog_description/meshes/wheel.stl" />
             </geometry>
             <material name="dark_grey" />
@@ -103,5 +103,5 @@
             <origin xyz="0 0 0" rpy="0 0 0"/>
             <geometry>
-            <mesh filename="model://warthog_description/meshes/tracks.dae" />
+            <mesh filename="package://warthog_description/meshes/tracks.dae" />
             </geometry>
             <material name="dark_grey" />
@@ -110,5 +110,5 @@
             <origin xyz="0 0 0" rpy="0 0 0"/>
             <geometry>
-            <mesh filename="model://warthog_description/meshes/tracks_collision.stl" />
+            <mesh filename="package://warthog_description/meshes/tracks_collision.stl" />
             </geometry>
         </collision>
@@ -197,5 +197,5 @@
             <origin xyz="0 0 0" rpy="0 0 0"/>
             <geometry>
-                <mesh filename="model://warthog_description/meshes/chassis.stl" />
+                <mesh filename="package://warthog_description/meshes/chassis.stl" />
             </geometry>
             <material name="black"><color rgba="0.15 0.15 0.15 1.0" /></material>
@@ -204,5 +204,5 @@
             <origin xyz="0 0 0" rpy="0 0 0"/>
             <geometry>
-                <mesh filename="model://warthog_description/meshes/e-stop.stl" />
+                <mesh filename="package://warthog_description/meshes/e-stop.stl" />
             </geometry>
             <material name="red"><color rgba="0.9 0.0 0.0 1.0" /></material>
@@ -211,5 +211,5 @@
             <origin xyz="0 0 0" rpy="0 0 0"/>
             <geometry>
-                <mesh filename="model://warthog_description/meshes/chassis-collision.stl" />
+                <mesh filename="package://warthog_description/meshes/chassis-collision.stl" />
             </geometry>
         </collision>
@@ -223,5 +223,5 @@
             <origin xyz="0 0 0" rpy="0 0 0"/>
             <geometry>
-                <mesh filename="model://warthog_description/meshes/diff-link.stl" />
+                <mesh filename="package://warthog_description/meshes/diff-link.stl" />
             </geometry>
             <material name="light_grey" />
@@ -230,5 +230,5 @@
             <origin xyz="0 0 0" rpy="0 0 0"/>
             <geometry>
-                <mesh filename="model://warthog_description/meshes/susp-link.stl" />
+                <mesh filename="package://warthog_description/meshes/susp-link.stl" />
             </geometry>
             <material name="light_grey" />
@@ -237,5 +237,5 @@
             <origin xyz="0 0 0" rpy="0 0 0"/>
             <geometry>
-                <mesh filename="model://warthog_description/meshes/susp-link.stl" />
+                <mesh filename="package://warthog_description/meshes/susp-link.stl" />
             </geometry>
             <material name="light_grey" />
@@ -262,5 +262,5 @@
             <origin xyz="0 0 0" rpy="0 0 ${side*PI/2}"/>
             <geometry>
-            <mesh filename="model://warthog_description/meshes/rocker.stl" />
+            <mesh filename="package://warthog_description/meshes/rocker.stl" />
             </geometry>
             <material name="black"><color rgba="0.15 0.15 0.15 1.0" /></material>
@@ -269,5 +269,5 @@
             <origin xyz="0 0 0" rpy="0 0 ${side*PI/2}"/>
             <geometry>
-            <mesh filename="model://warthog_description/meshes/fenders.stl" />
+            <mesh filename="package://warthog_description/meshes/fenders.stl" />
             </geometry>
             <material name="yellow"><color rgba="0.95 0.816 0.082 1.0" /></material>
@@ -276,5 +276,5 @@
             <origin xyz="0 0 0" rpy="0 0 ${side*PI/2}"/>
             <geometry>
-            <mesh filename="model://warthog_description/meshes/fenders-collision.stl" />
+            <mesh filename="package://warthog_description/meshes/fenders-collision.stl" />
             </geometry>
         </collision>
@@ -300,5 +300,5 @@
         <visual>
             <geometry>
-            <mesh filename="model://warthog_description/meshes/buttons.stl"/>
+            <mesh filename="package://warthog_description/meshes/buttons.stl"/>
             </geometry>
             <material name="red"><color rgba="0.9 0.0 0.0 1.0" /></material>
@@ -324,5 +324,5 @@
                 <material name="light_grey" />
                 <geometry>
-                <mesh filename="model://warthog_description/meshes/antenna_${prefix}.stl"/>
+                <mesh filename="package://warthog_description/meshes/antenna_${prefix}.stl"/>
                 </geometry>
             </visual>
@@ -348,5 +348,5 @@
                 <material name="light_grey"/>
                 <geometry>
-                    <mesh filename="model://warthog_description/meshes/antenna_estop.stl"/>
+                    <mesh filename="package://warthog_description/meshes/antenna_estop.stl"/>
                 </geometry>
                 </visual>
@@ -372,5 +372,5 @@
                 <origin xyz="0 ${side*-0.029} 0" rpy="0 0 0"/>
                 <geometry>
-                    <mesh filename="model://warthog_description/meshes/light.stl" />
+                    <mesh filename="package://warthog_description/meshes/light.stl" />
                 </geometry>
                 <material name="white"><color rgba="0.9 0.9 0.9 1.0" /></material>
@@ -379,5 +379,5 @@
                 <origin xyz="0 ${side*-0.022} 0" rpy="0 0 0"/>
                 <geometry>
-                <mesh filename="model://warthog_description/meshes/light-collision.stl" />
+                <mesh filename="package://warthog_description/meshes/light-collision.stl" />
                 </geometry>
                 <material name="white"><color rgba="0.9 0.9 0.9 1.0" /></material>
@@ -406,5 +406,5 @@
                 <origin xyz="0 ${side*-0.029} 0" rpy="0 0 ${side*PI}"/>
                 <geometry>
-                <mesh filename="model://warthog_description/meshes/light.stl" />
+                <mesh filename="package://warthog_description/meshes/light.stl" />
                 </geometry>
                 <material name="red"><color rgba="0.9 0.0 0.0 1.0" /></material>
@@ -413,5 +413,5 @@
                 <origin xyz="0 ${side*-0.022} 0" rpy="0 0 ${side*PI}"/>
                 <geometry>
-                <mesh filename="model://warthog_description/meshes/light-collision.stl" />
+                <mesh filename="package://warthog_description/meshes/light-collision.stl" />
                 </geometry>
                 <material name="red"><color rgba="0.9 0.0 0.0 1.0" /></material>
