Commit message: update urdf folder

File: warthog_description/urdf/warthog.urdf.xacro (robot description, xacro)
@@ -1,24 +1,6 @@
-<?xml version="1.0"?>
+<?xml version="1.0" ?>
 <robot name="warthog" xmlns:xacro="http://www.ros.org/wiki/xacro">
-    <xacro:property name="PI" value="3.1415926535897931"/>
-    <xacro:property name="wheel_radius" value="0.3" />
-    <xacro:property name="wheel_width" value="0.25" />
-    <xacro:property name="wheel_mass" value="15" />
-    <xacro:property name="wheel_to_track_ratio" value="0.5962" />
-    <xacro:property name="axle_x_offset" value="0.457367" />
-    <xacro:property name="axle_y_offset" value="0.0" />
-    <xacro:property name="axle_z_offset" value="-0.012977" />
-    <xacro:property name="diff_unit_length" value="1.34" />
-    <xacro:property name="diff_unit_width" value="0.28" />
-    <xacro:property name="diff_unit_height" value="0.63"/>
-    <xacro:property name="diff_unit_mass" value="50" />
-    <xacro:property name="diff_unit_offset_x" value="0.00" />
-    <xacro:property name="diff_unit_offset_y" value="0.56821" />
-    <xacro:property name="diff_unit_offset_z" value="0.0" />
-    <xacro:property name="chassis_length" value="1.35" />
-    <xacro:property name="chassis_width" value="0.70" />
-    <xacro:property name="chassis_height" value="0.30" />
-    <xacro:property name="chassis_mass" value="100" />
-    <xacro:property name="dummy_inertia" value="1e-09"/>
+    <xacro:include filename="$(find warthog_description)/urdf/base.xacro" />
+    <xacro:include filename="$(find warthog_description)/urdf/utils.xacro" />
     <!--
         Optional paint colors.
@@ -29,14 +11,4 @@
         - sand
     -->
-    <xacro:macro name="wheel_inertia" params="m r h">
-        <inertia ixx="${m*(3*r*r+h*h)/12}" ixy="0" ixz="0"
-                iyy="${m*r*r/2}" iyz="0"
-                izz="${m*(3*r*r+h*h)/12}" />
-    </xacro:macro>
-    <xacro:macro name="box_inertia" params="m x y z">
-        <inertia ixx="${m*(y*y+z*z)/12}" ixy="0" ixz="0"
-                iyy="${m*(x*x+z*z)/12}" iyz="0"
-                izz="${m*(x*x+z*z)/12}" />
-    </xacro:macro>
     <material name="dark_grey"><color rgba="0.2 0.2 0.2 1.0" /></material>
     <material name="light_grey"><color rgba="0.4 0.4 0.4 1.0" /></material>
@@ -45,131 +17,54 @@
     <material name="white"><color rgba="0.9 0.9 0.9 1.0" /></material>
     <material name="red"><color rgba="0.9 0.0 0.0 1.0" /></material>
-    <!-- ======================================================= -->
-    <!--                      Wheels                         -->
-    <!-- ======================================================= -->
-    <xacro:macro name="wheel" params="prefix side *joint_pose">
-        <link name="${prefix}_${side}_wheel_link">
-        <inertial>
-            <origin xyz="0 0 0" rpy="0 0 0" />
-            <mass value="${wheel_mass}" />
-            <xacro:wheel_inertia m="${wheel_mass}" r="${wheel_radius}" h="${wheel_width}" />
-        </inertial>
-        <visual>
-            <origin xyz="0 0 0" rpy="0 0 ${PI/2}"/>
-            <geometry>
-            <mesh filename="package://warthog_description/meshes/wheel.stl" />
-            </geometry>
-            <material name="dark_grey" />
-        </visual>
-        <collision>
-            <origin xyz="0 0 0" rpy="${PI/2} 0 0"/>
-            <geometry>
-            <cylinder radius="${wheel_radius}" length="${wheel_width}"/>
-            </geometry>
-        </collision>
-        </link>
-        <joint name="${prefix}_${side}_wheel_joint" type="continuous">
-            <parent link="${side}_diff_unit_link"/>
-            <child link="${prefix}_${side}_wheel_link"/>
-            <xacro:insert_block name="joint_pose" />
-            <axis xyz="0 1 0"/>
-        </joint>
-        <gazebo reference="${prefix}_${side}_wheel_link">
-            <selfCollide>false</selfCollide>
-            <mu1>0.5</mu1>
-            <mu2>0.5</mu2>
-            <kp value="10000000.0" />
-            <kd value="1.0" />
-            <fdir1 value="1 0 0" />
-            <material>Gazebo/DarkGrey</material>
-        </gazebo>
-        <transmission name="${prefix}_${side}_wheel_trans">
-            <type>transmission_interface/SimpleTransmission</type>
-            <joint name="${prefix}_${side}_wheel_joint">
-                <hardwareInterface>hardware_interface/VelocityJointInterface</hardwareInterface>
-            </joint>
-            <actuator name="${prefix}_${side}_actuator">
-                <hardwareInterface>hardware_interface/VelocityJointInterface</hardwareInterface>
-                <mechanicalReduction>1</mechanicalReduction>
-            </actuator>
-        </transmission>
-    </xacro:macro>
-    <!-- ======================================================= -->
-    <!--                       Tracks                          -->
-    <!-- ======================================================= -->
-    <xacro:macro name="track" params="prefix side *joint_pose">
-        <link name="${prefix}_${side}_track_link">
-        <visual>
-            <origin xyz="0 0 0" rpy="0 0 0"/>
-            <geometry>
-            <mesh filename="package://warthog_description/meshes/tracks.dae" />
-            </geometry>
-            <material name="dark_grey" />
-        </visual>
-        <collision>
-            <origin xyz="0 0 0" rpy="0 0 0"/>
-            <geometry>
-            <mesh filename="package://warthog_description/meshes/tracks_collision.stl" />
-            </geometry>
-        </collision>
-        </link>
-        <joint name="${prefix}_${side}_track_joint" type="fixed">
-            <parent link="${side}_diff_unit_link"/>
-            <child link="${prefix}_${side}_track_link"/>
-            <xacro:insert_block name="joint_pose" />
-            <axis xyz="0 1 0"/>
-        </joint>
-        <!-- This adds wheels that rotate instead of tracks. -->
-        <link name="${prefix}_${side}_wheel_link">
-        <collision>
-            <origin xyz="0 0 0" rpy="${PI/2} 0 0"/>
-            <geometry>
-            <cylinder radius="${wheel_radius*wheel_to_track_ratio}" length="${wheel_width}"/>
-            </geometry>
-        </collision>
-        </link>
-        <joint name="${prefix}_${side}_wheel_joint" type="continuous">
-            <parent link="${side}_diff_unit_link"/>
-            <child link="${prefix}_${side}_wheel_link"/>
-            <xacro:insert_block name="joint_pose" />
-            <axis xyz="0 1 0"/>
-        </joint>
-        <transmission name="${prefix}_${side}_wheel_trans">
-        <type>transmission_interface/SimpleTransmission</type>
-        <joint name="${prefix}_${side}_wheel_joint">
-            <hardwareInterface>hardware_interface/VelocityJointInterface</hardwareInterface>
-        </joint>
-        <actuator name="${prefix}_${side}_actuator">
-            <hardwareInterface>hardware_interface/VelocityJointInterface</hardwareInterface>
-            <mechanicalReduction>1</mechanicalReduction>
-        </actuator>
-        </transmission>
-    </xacro:macro>
     <xacro:unless value="$(optenv WARTHOG_TRACKS 0)">
         <xacro:wheel prefix="front" side="left">
-            <origin xyz="${axle_x_offset*1} ${axle_y_offset*1} ${axle_z_offset}" rpy="0 0 0" />
+            <origin
+                xyz="${axle_x_offset*1} ${axle_y_offset*1} ${axle_z_offset}"
+                rpy="0 0 0"
+            />
         </xacro:wheel>
         <xacro:wheel prefix="front" side="right">
-            <origin xyz="${axle_x_offset*1} ${axle_y_offset*-1} ${axle_z_offset}" rpy="0 0 0" />
+            <origin
+                xyz="${axle_x_offset*1} ${axle_y_offset*-1} ${axle_z_offset}"
+                rpy="0 0 0"
+            />
         </xacro:wheel>
         <xacro:wheel prefix="rear" side="left">
-            <origin xyz="${axle_x_offset*-1} ${axle_y_offset*1} ${axle_z_offset}" rpy="0 0 0" />
+            <origin
+                xyz="${axle_x_offset*-1} ${axle_y_offset*1} ${axle_z_offset}"
+                rpy="0 0 0"
+            />
         </xacro:wheel>
         <xacro:wheel prefix="rear" side="right">
-            <origin xyz="${axle_x_offset*-1} ${axle_y_offset*-1} ${axle_z_offset}" rpy="0 0 0" />
+            <origin
+                xyz="${axle_x_offset*-1} ${axle_y_offset*-1} ${axle_z_offset}"
+                rpy="0 0 0"
+            />
         </xacro:wheel>
     </xacro:unless>
     <xacro:if value="$(optenv WARTHOG_TRACKS 0)">
         <xacro:track prefix="front" side="left">
-            <origin xyz="${axle_x_offset*1} ${axle_y_offset*1} ${axle_z_offset}" rpy="0 0 0" />
+            <origin
+                xyz="${axle_x_offset*1} ${axle_y_offset*1} ${axle_z_offset}"
+                rpy="0 0 0"
+            />
         </xacro:track>
         <xacro:track prefix="front" side="right">
-            <origin xyz="${axle_x_offset*1} ${axle_y_offset*-1} ${axle_z_offset}" rpy="0 0 0" />
+            <origin
+                xyz="${axle_x_offset*1} ${axle_y_offset*-1} ${axle_z_offset}"
+                rpy="0 0 0"
+            />
         </xacro:track>
         <xacro:track prefix="rear" side="left">
-            <origin xyz="${axle_x_offset*-1} ${axle_y_offset*1} ${axle_z_offset}" rpy="0 0 ${PI}" />
+            <origin
+                xyz="${axle_x_offset*-1} ${axle_y_offset*1} ${axle_z_offset}"
+                rpy="0 0 ${PI}"
+            />
         </xacro:track>
         <xacro:track prefix="rear" side="right">
-            <origin xyz="${axle_x_offset*-1} ${axle_y_offset*-1} ${axle_z_offset}" rpy="0 0 ${PI}" />
+            <origin
+                xyz="${axle_x_offset*-1} ${axle_y_offset*-1} ${axle_z_offset}"
+                rpy="0 0 ${PI}"
+            />
         </xacro:track>
     </xacro:if>
@@ -177,8 +72,8 @@
     <!--                       BASE                          -->
     <!-- ======================================================= -->
-    <link name="base_link"></link>
+    <link name="base_link" />
     <joint name="base_link_joint" type="fixed">
         <origin xyz="0 0 0.025" rpy="0 0 0" />
-        <parent link="base_link"/>
+        <parent link="base_link" />
         <child link="chassis_link" />
     </joint>
@@ -189,27 +84,39 @@
     <link name="chassis_link">
         <inertial>
-            <origin xyz="0 0 0" rpy="0 0 0"/>
-            <mass value="${chassis_mass}"/>
-            <xacro:box_inertia m="${chassis_mass}" x="${chassis_length}"
-                            y="${chassis_width}" z="${chassis_height}" />
+            <origin xyz="0 0 0" rpy="0 0 0" />
+            <mass value="${chassis_mass}" />
+            <xacro:box_inertia
+                m="${chassis_mass}"
+                x="${chassis_length}"
+                y="${chassis_width}"
+                z="${chassis_height}"
+            />
         </inertial>
         <visual>
-            <origin xyz="0 0 0" rpy="0 0 0"/>
-            <geometry>
-                <mesh filename="package://warthog_description/meshes/chassis.stl" />
-            </geometry>
-            <material name="black"><color rgba="0.15 0.15 0.15 1.0" /></material>
-        </visual>
-        <visual>
-            <origin xyz="0 0 0" rpy="0 0 0"/>
-            <geometry>
-                <mesh filename="package://warthog_description/meshes/e-stop.stl" />
+            <origin xyz="0 0 0" rpy="0 0 0" />
+            <geometry>
+                <mesh
+                    filename="package://warthog_description/meshes/chassis.stl"
+                />
+            </geometry>
+            <material name="black"><color
+                    rgba="0.15 0.15 0.15 1.0"
+                /></material>
+        </visual>
+        <visual>
+            <origin xyz="0 0 0" rpy="0 0 0" />
+            <geometry>
+                <mesh
+                    filename="package://warthog_description/meshes/e-stop.stl"
+                />
             </geometry>
             <material name="red"><color rgba="0.9 0.0 0.0 1.0" /></material>
         </visual>
         <collision>
-            <origin xyz="0 0 0" rpy="0 0 0"/>
-            <geometry>
-                <mesh filename="package://warthog_description/meshes/chassis-collision.stl" />
+            <origin xyz="0 0 0" rpy="0 0 0" />
+            <geometry>
+                <mesh
+                    filename="package://warthog_description/meshes/chassis-collision.stl"
+                />
             </geometry>
         </collision>
@@ -221,21 +128,27 @@
     <link name="diff_link">
         <visual>
-            <origin xyz="0 0 0" rpy="0 0 0"/>
-            <geometry>
-                <mesh filename="package://warthog_description/meshes/diff-link.stl" />
+            <origin xyz="0 0 0" rpy="0 0 0" />
+            <geometry>
+                <mesh
+                    filename="package://warthog_description/meshes/diff-link.stl"
+                />
             </geometry>
             <material name="light_grey" />
         </visual>
         <visual>
-            <origin xyz="0 0 0" rpy="0 0 0"/>
-            <geometry>
-                <mesh filename="package://warthog_description/meshes/susp-link.stl" />
+            <origin xyz="0 0 0" rpy="0 0 0" />
+            <geometry>
+                <mesh
+                    filename="package://warthog_description/meshes/susp-link.stl"
+                />
             </geometry>
             <material name="light_grey" />
         </visual>
         <visual>
-            <origin xyz="0 0 0" rpy="0 0 0"/>
-            <geometry>
-                <mesh filename="package://warthog_description/meshes/susp-link.stl" />
+            <origin xyz="0 0 0" rpy="0 0 0" />
+            <geometry>
+                <mesh
+                    filename="package://warthog_description/meshes/susp-link.stl"
+                />
             </geometry>
             <material name="light_grey" />
@@ -244,212 +157,11 @@
     <!-- Joint to attach the diff link to the chassis -->
     <joint name="diff_link_joint" type="fixed">
-        <parent link="chassis_link"/>
-        <child link="diff_link"/>
+        <parent link="chassis_link" />
+        <child link="diff_link" />
         <origin xyz="-0.5826 0 0.24979" rpy="0 0 0" />
     </joint>
-    <!-- ======================================================= -->
-    <!--                       Diff Unit                        -->
-    <!-- ======================================================= -->
-    <xacro:macro name="diff_unit" params="prefix side">
-        <link name="${prefix}_diff_unit_link">
-        <inertial>
-            <origin xyz="0 ${side*-1*0.05} 0.197" rpy="0 0 0"/>
-            <mass value="${diff_unit_mass}"/>
-            <xacro:box_inertia m="${diff_unit_mass}" x="${diff_unit_length}"
-                            y="${diff_unit_width}" z="${diff_unit_height}" />
-        </inertial>
-        <visual>
-            <origin xyz="0 0 0" rpy="0 0 ${side*PI/2}"/>
-            <geometry>
-            <mesh filename="package://warthog_description/meshes/rocker.stl" />
-            </geometry>
-            <material name="black"><color rgba="0.15 0.15 0.15 1.0" /></material>
-        </visual>
-        <visual>
-            <origin xyz="0 0 0" rpy="0 0 ${side*PI/2}"/>
-            <geometry>
-            <mesh filename="package://warthog_description/meshes/fenders.stl" />
-            </geometry>
-            <material name="yellow"><color rgba="0.95 0.816 0.082 1.0" /></material>
-        </visual>
-        <collision>
-            <origin xyz="0 0 0" rpy="0 0 ${side*PI/2}"/>
-            <geometry>
-            <mesh filename="package://warthog_description/meshes/fenders-collision.stl" />
-            </geometry>
-        </collision>
-        <collision>
-            <origin xyz="0.0 ${-side*0.02} 0.52" rpy="0 0 ${side*PI/2}"/>
-            <geometry>
-            <box size="0.28 0.95 0.024"/>
-            </geometry>
-        </collision>
-        </link>
-        <joint name="${prefix}_diff_unit_joint" type="fixed">
-            <limit upper="0.4" lower="-0.4" effort="100" velocity="1"/>
-            <parent link="chassis_link"/>
-            <child link="${prefix}_diff_unit_link"/>
-            <origin xyz="${diff_unit_offset_x} ${diff_unit_offset_y*side} ${diff_unit_offset_z}" rpy="0 0 0" />
-            <axis xyz="0 1 0"/>
-            <dynamics damping="100" friction="0.5"/>
-        </joint>
-        <!-- ======================================================= -->
-        <!--                       Diff Unit Buttons                -->
-        <!-- ======================================================= -->
-        <link name="${prefix}_diff_unit_buttons_link">
-        <visual>
-            <geometry>
-            <mesh filename="package://warthog_description/meshes/buttons.stl"/>
-            </geometry>
-            <material name="red"><color rgba="0.9 0.0 0.0 1.0" /></material>
-        </visual>
-        <collision>
-            <origin xyz="0.0395 0.4315 0.520" rpy="0 0 0"/>
-            <geometry>
-            <cylinder radius="0.0205" length="0.014"/>
-            </geometry>
-        </collision>
-        <collision>
-            <origin xyz="0.0395 -0.4315 0.520" rpy="0 0 0"/>
-            <geometry>
-            <cylinder radius="0.0205" length="0.014"/>
-            </geometry>
-        </collision>
-        </link>
-        <!-- ======================================================= -->
-        <!--                Wi-Fi and Controller Antenna             -->
-        <!-- ======================================================= -->
-        <link name="${prefix}_diff_unit_antenna_link">
-            <visual>
-                <material name="light_grey" />
-                <geometry>
-                <mesh filename="package://warthog_description/meshes/antenna_${prefix}.stl"/>
-                </geometry>
-            </visual>
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