Commit message: add urdf files

File: warthog_description/urdf/warthog.urdf.xacro (robot description, xacro)
@@ -1,6 +1,25 @@
 <?xml version="1.0" ?>
 <robot name="warthog" xmlns:xacro="http://www.ros.org/wiki/xacro">
-    <xacro:include filename="$(find warthog_description)/urdf/base.xacro" />
+    <xacro:include
+        filename="$(find warthog_description)/urdf/wheel.urdf.xacro"
+    />
+    <xacro:include
+        filename="$(find warthog_description)/urdf/diff_unit.urdf.xacro"
+    />
     <xacro:include filename="$(find warthog_description)/urdf/utils.xacro" />
+    <xacro:include
+        filename="$(find warthog_description)/urdf/gazebo.urdf.xacro"
+    />
+    <xacro:include
+        filename="$(find warthog_description)/urdf/ros2_control.urdf.xacro"
+    />
+    <xacro:include
+        filename="$(find warthog_description)/urdf/body.urdf.xacro"
+    />
+    <!-- <xacro:property name="dummy_inertia" value="1e-09" /> -->
+    <xacro:property name="PI" value="3.1415926535897931" />
+    <xacro:property name="axle_x_offset" value="0.457367" />
+    <xacro:property name="axle_y_offset" value="0.0" />
+    <xacro:property name="axle_z_offset" value="-0.012977" />
     <!--
         Optional paint colors.
@@ -69,154 +88,7 @@
         </xacro:track>
     </xacro:if>
-    <!-- ======================================================= -->
-    <!--                       BASE                          -->
-    <!-- ======================================================= -->
-    <link name="base_link" />
-    <joint name="base_link_joint" type="fixed">
-        <origin xyz="0 0 0.025" rpy="0 0 0" />
-        <parent link="base_link" />
-        <child link="chassis_link" />
-    </joint>
-  <!-- ======================================================= -->
-  <!--                       Chassis                          -->
-  <!-- ======================================================= -->
-   <!-- Chassis link (black part) -->
-    <link name="chassis_link">
-        <inertial>
-            <origin xyz="0 0 0" rpy="0 0 0" />
-            <mass value="${chassis_mass}" />
-            <xacro:box_inertia
-                m="${chassis_mass}"
-                x="${chassis_length}"
-                y="${chassis_width}"
-                z="${chassis_height}"
-            />
-        </inertial>
-        <visual>
-            <origin xyz="0 0 0" rpy="0 0 0" />
-            <geometry>
-                <mesh
-                    filename="package://warthog_description/meshes/chassis.stl"
-                />
-            </geometry>
-            <material name="black"><color
-                    rgba="0.15 0.15 0.15 1.0"
-                /></material>
-        </visual>
-        <visual>
-            <origin xyz="0 0 0" rpy="0 0 0" />
-            <geometry>
-                <mesh
-                    filename="package://warthog_description/meshes/e-stop.stl"
-                />
-            </geometry>
-            <material name="red"><color rgba="0.9 0.0 0.0 1.0" /></material>
-        </visual>
-        <collision>
-            <origin xyz="0 0 0" rpy="0 0 0" />
-            <geometry>
-                <mesh
-                    filename="package://warthog_description/meshes/chassis-collision.stl"
-                />
-            </geometry>
-        </collision>
-    </link>
-  <!-- ======================================================= -->
-  <!--                       Diff Link                         -->
-  <!-- this is only for put the floating diff in the robot     -->
-  <!-- ======================================================= -->
-    <link name="diff_link">
-        <visual>
-            <origin xyz="0 0 0" rpy="0 0 0" />
-            <geometry>
-                <mesh
-                    filename="package://warthog_description/meshes/diff-link.stl"
-                />
-            </geometry>
-            <material name="light_grey" />
-        </visual>
-        <visual>
-            <origin xyz="0 0 0" rpy="0 0 0" />
-            <geometry>
-                <mesh
-                    filename="package://warthog_description/meshes/susp-link.stl"
-                />
-            </geometry>
-            <material name="light_grey" />
-        </visual>
-        <visual>
-            <origin xyz="0 0 0" rpy="0 0 0" />
-            <geometry>
-                <mesh
-                    filename="package://warthog_description/meshes/susp-link.stl"
-                />
-            </geometry>
-            <material name="light_grey" />
-        </visual>
-    </link>
-    <!-- Joint to attach the diff link to the chassis -->
-    <joint name="diff_link_joint" type="fixed">
-        <parent link="chassis_link" />
-        <child link="diff_link" />
-        <origin xyz="-0.5826 0 0.24979" rpy="0 0 0" />
-    </joint>
     <!-- instancia de unidad diferencial -->
     <xacro:diff_unit prefix="left" side="1" />
     <xacro:diff_unit prefix="right" side="-1" />
-    <ros2_control name="GazeboSimSystem" type="system">
-    <hardware>
-        <plugin>ign_ros2_control/IgnitionSystem</plugin>
-    </hardware>
-    <joint name="front_left_wheel_joint">
-        <command_interface name="velocity">
-        <param name="min">-1</param>
-        <param name="max">1</param>
-        </command_interface>
-        <state_interface name="position" />
-        <state_interface name="velocity" />
-    </joint>
-    <joint name="front_right_wheel_joint">
-        <command_interface name="velocity">
-        <param name="min">-1</param>
-        <param name="max">1</param>
-        </command_interface>
-        <state_interface name="position" />
-        <state_interface name="velocity" />
-    </joint>
-    <joint name="rear_left_wheel_joint">
-        <command_interface name="velocity">
-        <param name="min">-1</param>
-        <param name="max">1</param>
-        </command_interface>
-        <state_interface name="position" />
-        <state_interface name="velocity" />
-    </joint>
-    <joint name="rear_right_wheel_joint">
-        <command_interface name="velocity">
-        <param name="min">-1</param>
-        <param name="max">1</param>
-        </command_interface>
-        <state_interface name="position" />
-        <state_interface name="velocity" />
-    </joint>
-    </ros2_control>
-    <gazebo>
-      <plugin
-            filename="ignition-gazebo-sensors-system"
-            name="ignition::gazebo::systems::Sensors"
-        >
-        <render_engine>ogre</render_engine>
-      </plugin>
-      <plugin
-            filename="ign_ros2_control-system"
-            name="ign_ros2_control::IgnitionROS2ControlPlugin"
-        >
-        <ros>
-            <namespace>warthog</namespace>
-            <!-- <remapping>/warthog/diff_drive_base_controller/cmd_vel:=cmd_vel</remapping> -->
-        </ros>
-        <parameters>$(find warthog_bringup)/config/controllers.yaml</parameters>
-      </plugin>
-    </gazebo>
     <!-- sudo apt install ros-humble-ros2-controllers ros-humble-ros2-control sudo apt-get install ros-humble-ign-ros2-control-->
 </robot>
